Commit message: Add ROS camera to sd5

File: models/rotors_description/urdf/sd5_base.xacro (robot description, xacro)
@@ -47,4 +47,22 @@
   </xacro:mavlink_interface_macro>
   </xacro:if>
+  <xacro:camera_macro
+    namespace="${namespace}"
+    parent_link="base_link"
+    camera_suffix="sd5"
+    frame_rate="30.0"
+    horizontal_fov="1.3962634"
+    image_width="800"
+    image_height="800"
+    image_format="R8G8B8"
+    min_distance="0.02"
+    max_distance="300"
+    noise_mean="0.0"
+    noise_stddev="0.007"
+    enable_visual="1"
+    >
+    <box size="0.05 0.05 0.05" />
+    <origin xyz="0 0 0.07" rpy="0 0 0" />
+  </xacro:camera_macro>
   <!-- Mount an ADIS16448 IMU. -->
   <xacro:imu_plugin_macro

Commit message: Mount two ROS cameras to sd5

File: models/rotors_description/urdf/sd5_base.xacro (robot description, xacro)
@@ -50,5 +50,5 @@
     namespace="${namespace}"
     parent_link="base_link"
-    camera_suffix="sd5"
+    camera_suffix="sd5_left"
     frame_rate="30.0"
     horizontal_fov="1.3962634"
@@ -63,5 +63,23 @@
     >
     <box size="0.05 0.05 0.05" />
-    <origin xyz="0 0 0.07" rpy="0 0 0" />
+    <origin xyz="0.05 0.025 0.07" rpy="0 0 0" />
+  </xacro:camera_macro>
+  <xacro:camera_macro
+    namespace="${namespace}"
+    parent_link="base_link"
+    camera_suffix="sd5_right"
+    frame_rate="30.0"
+    horizontal_fov="1.3962634"
+    image_width="800"
+    image_height="800"
+    image_format="R8G8B8"
+    min_distance="0.02"
+    max_distance="300"
+    noise_mean="0.0"
+    noise_stddev="0.007"
+    enable_visual="1"
+    >
+    <box size="0.05 0.05 0.05" />
+    <origin xyz="0.05 -0.025 0.07" rpy="0 0 0" />
   </xacro:camera_macro>
   <!-- Mount an ADIS16448 IMU. -->

Commit message: add rear camera

File: models/rotors_description/urdf/sd5_base.xacro (robot description, xacro)
@@ -83,4 +83,22 @@
     <origin xyz="0.05 -0.025 0.07" rpy="0 0 0" />
   </xacro:camera_macro>
+  <xacro:camera_macro
+    namespace="${namespace}"
+    parent_link="base_link"
+    camera_suffix="sd5_rear"
+    frame_rate="30.0"
+    horizontal_fov="1.3962634"
+    image_width="800"
+    image_height="800"
+    image_format="R8G8B8"
+    min_distance="0.02"
+    max_distance="300"
+    noise_mean="0.0"
+    noise_stddev="0.007"
+    enable_visual="1"
+    >
+    <box size="0.02 0.02 0.02" />
+    <origin xyz="-0.07 0 -0.04" rpy="0 1.57079632679 0" />
+  </xacro:camera_macro>
   <!-- Mount an ADIS16448 IMU. -->
   <xacro:imu_plugin_macro

Commit message: adjust camera dimensions to mock zed camera

File: models/rotors_description/urdf/sd5_base.xacro (robot description, xacro)
@@ -62,6 +62,6 @@
     enable_visual="1"
     >
-    <box size="0.05 0.05 0.05" />
-    <origin xyz="0.05 0.025 0.07" rpy="0 0 0" />
+    <box size="0.03302 0.065532 0.029972" />
+    <origin xyz="0.05 0.054737 0.06" rpy="0 0 0" />
   </xacro:camera_macro>
   <xacro:camera_macro
@@ -80,6 +80,6 @@
     enable_visual="1"
     >
-    <box size="0.05 0.05 0.05" />
-    <origin xyz="0.05 -0.025 0.07" rpy="0 0 0" />
+    <box size="0.03302 0.065532 0.029972" />
+    <origin xyz="0.05 -0.054737 0.06" rpy="0 0 0" />
   </xacro:camera_macro>
   <xacro:camera_macro

Commit message: move cameras 2 cm forward and position lenses 12 cm apart

File: models/rotors_description/urdf/sd5_base.xacro (robot description, xacro)
@@ -63,5 +63,5 @@
     >
     <box size="0.03302 0.065532 0.029972" />
-    <origin xyz="0.05 0.054737 0.06" rpy="0 0 0" />
+    <origin xyz="0.07 0.06 0.06" rpy="0 0 0" />
   </xacro:camera_macro>
   <xacro:camera_macro
@@ -81,5 +81,5 @@
     >
     <box size="0.03302 0.065532 0.029972" />
-    <origin xyz="0.05 -0.054737 0.06" rpy="0 0 0" />
+    <origin xyz="0.07 -0.06 0.06" rpy="0 0 0" />
   </xacro:camera_macro>
   <xacro:camera_macro
